File: hardware/kicad/PicoFault.kicad_pcb (KiCad board)
At the start: 2 copper layers, 78 parts, among them J10 TRIGGER_VREF, J3 Conn_01x10, J4 Header 2, J5 Header 4, J6 Input Power:2x AA Battery, J7 GLITCHER_EN, J8 ANALOG_PINS, J9 TRIGGER_IN, Q1 AO3422, Q2 AO3422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

Commit message: Minor touch-ups
Parts:
- moved U5 14.4 mm to (147.3, 107.0)
Changed lines of the file:
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@@
 	(footprint "Package_TO_SOT_SMD:SOT-23-5"
 		(layer "F.Cu")
-		(at 132.955 105.455)
+		(at 147.3 107)
 		(descr "SOT, 5 Pin (JEDEC MO-178 Var AA https://www.jedec.org/document_search?search_api_views_fulltext=MO-178)")
 		(tags "SOT TO_SOT_SMD")
