File: hardware/kicad/PicoFault.kicad_sch (KiCad schematic)
At the start: 0 parts

Commit message: KiCAD initial commit
Parts:
- added C1, C3: 4.7uF, Capacitor_SMD:C_0805_2012Metric, symbol Device:C
- added C10, C8: 27pF, Capacitor_SMD:C_0603_1608Metric, symbol Device:C_Small
- added C11, C12, C14, C15, C16, C17, C18, C19, C20, C7: 100nF, Capacitor_SMD:C_0402_1005Metric, symbol Device:C_Small
- added C13, C9: 1uF, Capacitor_SMD:C_0603_1608Metric, symbol Device:C_Small
- added C2: 100nF, Capacitor_SMD:C_0603_1608Metric, symbol Device:C
- added C21, C22: 100nF, Capacitor_SMD:C_0603_1608Metric, symbol Device:C_Small
- added C23, C24, C5, C6: 10uF, Capacitor_SMD:C_0402_1005Metric, symbol Device:C_Small
- added C4: 0.47uF, BuggyCat:CAPC6153X500N, symbol Device:C
- added D1, D10, D2, D3: SM4005PL-TP, Diode_SMD:D_SOD-123F, symbol Diode:SM4005
- added D4: MURA160T3G, Diode_SMD:D_SMA, symbol Diode:SM4005
- added D5: MM3Zxx, Diode_SMD:D_SOD-323F, symbol Diode:MM3Zxx
- added D6: MBR120, Diode_SMD:D_SOD-123, symbol Diode:MBR340
- added D7: H.V.Detected, LED_SMD:LED_0603_1608Metric, symbol Device:LED
- added D8: Status, LED_SMD:LED_0603_1608Metric, symbol Device:LED
- added D9: Charge On, LED_SMD:LED_0603_1608Metric, symbol Device:LED
- added F1: 0.5A, Fuse:Fuse_0805_2012Metric, symbol Device:Fuse_Small
- added J1: Antenna, BuggyCat:732511150, symbol CatSniffer-rescue:Conn_Coaxial-Connector-CatStick-rescue-CatSniffer-rescue
- added J10: TRIGGER_VREF, Connector_PinSocket_2.54mm:PinSocket_1x02_P2.54mm_Vertical, symbol Connector:Conn_01x02_Pin
- added J2: BG306-02-A-2-0400-L-G, BuggyCat:BG30602A20400LG, symbol Connector:Screw_Terminal_01x02
- added J3: Conn_01x10, Connector_PinSocket_2.54mm:PinSocket_1x10_P2.54mm_Vertical, symbol Connector_Generic:Conn_01x10
- added J4: Header 2, Connector_PinHeader_2.54mm:PinHeader_1x02_P2.54mm_Vertical, symbol Connector_Generic:Conn_01x02
- added J5: Header 4, Connector_PinHeader_2.54mm:PinHeader_1x04_P2.54mm_Vertical, symbol Connector_Generic:Conn_01x04
- added J6: Input Power:2x AA Battery, Connector_PinHeader_2.54mm:PinHeader_1x02_P2.54mm_Vertical, symbol Connector_Generic:Conn_01x02
- added J7: GLITCHER_EN, Connector_PinSocket_2.54mm:PinSocket_1x02_P2.54mm_Vertical, symbol Connector:Conn_01x02_Pin
- added J8: ANALOG_PINS, Connector_PinSocket_2.54mm:PinSocket_1x02_P2.54mm_Vertical, symbol Connector:Conn_01x02_Pin
- added J9: TRIGGER_IN, Connector_PinSocket_2.54mm:PinSocket_1x02_P2.54mm_Vertical, symbol Connector:Conn_01x02_Pin
- added P1: USB_C_Plug_USB2.0, Connectors:C393939, symbol Connector:USB_C_Plug_USB2.0
- added Q1, Q2: AO3422, Package_TO_SOT_SMD:SOT-23, symbol Transistor_FET:AO3400A
- added Q3: LDA111STR, BuggyCat:SOP254P952X470-6N, symbol LDA111STR:LDA111STR
- added Q4: RGT16BM65DTL, Package_TO_SOT_SMD:TO-252-3_TabPin2, symbol IRLML0060TRPBF:IRLML0060TRPBF
- added Q5: DMG3415U-7, Package_TO_SOT_SMD:SOT-23, symbol Device:Q_PMOS_GSD
- added Q7: IRLML2502, Package_TO_SOT_SMD:SOT-23, symbol pico-glitcher:NMOSFETSOT23-GSD
- added Q8: IRF7807PBF, BuggyCat:SOIC-8_SI, symbol pico-glitcher:MOSFET-NCHANNEL-SOIC8
- added R1, R9: 10R, Resistor_SMD:R_0603_1608Metric, symbol Device:R
- added R10: 20M, Resistor_SMD:R_2010_5025Metric, symbol Device:R
- added R11: 300K, BuggyCat:RESC6432X120N, symbol Device:R
- added R12: 100K, Resistor_SMD:R_0603_1608Metric, symbol Device:R_Small
- added R13, R14, R16, R5, R6: 1K, Resistor_SMD:R_0603_1608Metric, symbol Device:R
- added R15: 4.7k, Resistor_SMD:R_0603_1608Metric, symbol Device:R
- added R17: 10K, Resistor_SMD:R_0603_1608Metric, symbol Device:R_Small
- added R18: 1k, Resistor_SMD:R_0603_1608Metric, symbol Device:R_Small
- added R19, R20: 27, Resistor_SMD:R_0603_1608Metric, symbol Device:R_Small
- added R2, R4: 5.1K, Resistor_SMD:R_0603_1608Metric, symbol Device:R
- added R21: 10k, Resistor_SMD:R_0603_1608Metric, symbol Device:R
- added R23, R24: 1R, Resistor_SMD:R_0603_1608Metric, symbol Device:R
- added R25, R26: 10K, Resistor_SMD:R_0603_1608Metric, symbol Device:R
- added R3: 75R, Resistor_SMD:R_0805_2012Metric, symbol Device:R
- added R7: 22K, Resistor_SMD:R_0603_1608Metric, symbol Device:R
- added R8: 2K, Resistor_SMD:R_0805_2012Metric, symbol Device:R
- added SW1, SW3, SW6: TL3305AF260QG, BuggyCat:TL3305AF160QG, symbol Switch:SW_Push
- added SW2: ON, chipshouter:OS102011MA1QN1, symbol Switch:SW_SPST
- added SW4: RESET, Button_Switch_SMD:SW_SPST_TL3342, symbol Switch:SW_Push
- added SW5: BOOT, Button_Switch_SMD:SW_SPST_TL3342, symbol Switch:SW_Push
- added SW7: SW_SP3T, BuggyCat:Sw3P1T, symbol Switch:SW_SP3T
- added T1, T2: ATB322524, BuggyCat:ATB3225240110T000, symbol Device:Transformer_1P_1S
- added U1: AP2112K-3.3, Package_TO_SOT_SMD:SOT-23-5, symbol HunterCat-NFC-rescue:AP2112K-3.3-Regulator_Linear
- added U2: W25Q16JV, BuggyCat:W25Q16JVUUIQ, symbol Memory_Flash:W25Q32JVZP
- added U3: RP2040, BuggyCat:RP2040-QFN-56, symbol PicoWAN-rescue:RP2040-MCU_RaspberryPi_and_Boards-PicoWAN-rescue-PicoWAN-rescue
- added U4: TXS0108EPW, Package_SO:TSSOP-20_4.4x6.5mm_P0.65mm, symbol Logic_LevelTranslator:TXS0108EPW
- added U5: TLV75718PDBV, Package_TO_SOT_SMD:SOT-23-5, symbol Regulator_Linear:TLV75718PDBV
- added U6: SN74LVC1T45DBV, Package_TO_SOT_SMD:SOT-23-6, symbol Logic_LevelTranslator:SN74LVC1T45DBV
- added Y1: 12Mhz, Crystal:Crystal_SMD_5032-2Pin_5.0x3.2mm, symbol Device:Crystal_Small
Connections:
- new net: C8.1, U3.20 (XIN), Y1.1
- new net: R18.2, U3.21 (XOUT)
- new net: D6.1 (K), Q5.2 (S), SW2.1 (A)
- new net: D1.1 (K), R1.1, R3.1
- new net: C2.1, R1.2, T1.4 (AA)
- new net: C1.1, C3.1, R3.2, T2.4 (AA)
- new net: D8.2 (A), R14.1
- new net: C10.1, R18.1, Y1.2
- new net: R21.2, U6.5 (DIR)
- new net: F1.1, P1.A4 (VBUS), P1.A9 (VBUS), P1.B4 (VBUS), P1.B9 (VBUS)
- new net: D10.2 (A), J6.1 (Pin_1)
- new net: Q1.3 (D), T2.1 (AB)
- new net: D4.2 (A), T2.2 (SA)
- new net: C4.2, D5.2 (A), J2.1 (Pin_1), Q3.2 (K), Q4.2, R8.2, SW1.1, T1.2 (SA), T2.3 (SB)
- new net: D7.2 (A), R13.1
- new net: P1.A5 (CC), R2.1
- new net: P1.B5 (VCONN), R4.1
- new net: D5.1 (K), Q4.1, R9.2
- new net: J1.2 (Ext), Q4.3
- new net: Q8.4 (G), R24.2, R26.2
- new net: R8.1, R9.1, T1.3 (SB)
- new net: R15.2, U4.10 (OE)
- new net: C4.1, D4.1 (K), J1.1 (In), R11.2
- new net: J3.2 (Pin_2), U4.1 (A1)
- new net: J3.3 (Pin_3), U4.3 (A2)
- new net: J3.4 (Pin_4), U4.4 (A3)
- new net: J3.5 (Pin_5), U4.5 (A4)
- new net: J3.6 (Pin_6), U4.6 (A5)
- new net: J3.7 (Pin_7), U4.7 (A6)
- new net: J3.8 (Pin_8), U4.8 (A7)
- new net: J3.9 (Pin_9), U4.9 (A8)
- new net: Q7.1 (G), R23.1, R25.1
- new net: D9.2 (A), R16.2
- new net: D2.1 (K), Q2.1 (G), R5.1
- new net: Q2.3 (D), T1.1 (AB)
- new net: D3.1 (K), Q1.1 (G), R6.1
- new net: J2.2 (Pin_2), R10.2, R11.1, SW1.2
- new net: Q3.1 (A), R10.1
- new net +: R19.2, U3.47 (USB_DP)
- new net +1V2: C11.1, C12.1, C9.1, U3.23 (DVDD), U3.45 (VREG_VOUT), U3.50 (DVDD)
- new net +1V8: C23.1, SW7.1, U5.5 (OUT)
- new net +3V3: C13.1, C14.1, C15.1, C16.1, C17.1, C18.1, C19.1, C20.1, C21.2, C6.1, C7.1, D1.2 (A), J5.2 (Pin_2), R17.1, R7.1, SW6.2, SW7.2, U1.5 (VOUT), U2.8 (VCC), U3.1 (IOVDD), U3.10 (IOVDD), U3.22 (IOVDD), U3.33 (IOVDD), U3.42 (IOVDD), U3.43 (ADC_AVDD), U3.44 (VREG_IN), U3.48 (USB_VDD), U3.49 (IOVDD), U4.19 (VCCB), U6.1 (VCCA)
- new net -: R20.2, U3.46 (USB_DM)
- new net ANALOG: J8.1 (Pin_1), J8.2 (Pin_2), U3.41 (GPIO29_ADC3)
- new net CHARGED: J5.1 (Pin_1), Q3.5 (C), R7.2, U3.29 (GPIO18), U3.38 (GPIO26_ADC0)
- new net D+: P1.A6 (D+), R19.1
- new net D-: P1.A7 (D-), R20.1
- new net GLITCHER: J7.1 (Pin_1), J7.2 (Pin_2), Q7.3 (D), Q8.5 (D@4), Q8.6 (D@3), Q8.7 (D@2), Q8.8 (D@1)
- new net GND: C1.2, C10.2, C11.2, C12.2, C13.2, C14.2, C15.2, C16.2, C17.2, C18.2, C19.2, C2.2, C20.2, C21.1, C22.2, C23.2, C24.2, C3.2, C5.2, C6.2, C7.2, C8.2, C9.2, D7.1 (K), D8.1 (K), D9.1 (K), J3.10 (Pin_10), J4.1 (Pin_1), J5.3 (Pin_3), J6.2 (Pin_2), P1.A1 (GND), P1.A12 (GND), P1.B1 (GND), P1.B12 (GND), P1.S1 (SHIELD), Q1.2 (S), Q2.2 (S), Q3.4 (E), Q7.2 (S), Q8.1 (S@1), Q8.2 (S@2), Q8.3 (S@3), R12.2, R2.2, R21.1, R25.2, R26.1, R4.2, R5.2, R6.2, SW3.1, SW4.1, SW5.1, U1.2 (GND), U2.4 (GND), U3.19 (TESTEN), U3.57 (GND), U4.11 (GND), U5.2 (GND), U6.2 (GND)
- new net GP0: U3.2 (GPIO0), U4.20 (B1)
- new net GP1: U3.3 (GPIO1), U4.18 (B2)
- new net GP10: R14.2, U3.13 (GPIO10)
- new net GP11: SW3.2, U3.14 (GPIO11)
- new net GP2: U3.4 (GPIO2), U4.17 (B3)
- new net GP27: R16.1, U3.39 (GPIO27_ADC1)
- new net GP28: SW6.1, U3.40 (GPIO28_ADC2)
- new net GP3: U3.5 (GPIO3), U4.16 (B4)
- new net GP4: U3.6 (GPIO4), U4.15 (B5)
- new net GP5: U3.7 (GPIO5), U4.14 (B6)
- new net GP6: U3.8 (GPIO6), U4.13 (B7)
- new net GP7: U3.9 (GPIO7), U4.12 (B8)
- new net GP9: R13.2, U3.12 (GPIO9)
- new net HPGLITCH2: R24.1, U3.27 (GPIO16)
- new net HVPULSE: D2.2 (A), J4.2 (Pin_2), U3.17 (GPIO14)
- new net HVPWM: D3.2 (A), J5.4 (Pin_4), U3.31 (GPIO20)
- new net LPGLITCH2: R23.2, U3.28 (GPIO17)
- new net QSPI_CS: R17.2, SW5.2, U2.1 (~{CS}), U3.56 (QSPI_SS)
- new net QSPI_DATA0: U2.5 (DI(IO0)), U3.53 (QSPI_SD0)
- new net QSPI_DATA1: U2.2 (DO(IO1)), U3.55 (QSPI_SD1)
- new net QSPI_DATA2: U2.3 (IO2), U3.54 (QSPI_SD2)
- new net QSPI_DATA3: U2.7 (IO3), U3.51 (QSPI_SD3)
- new net QSPI_SCK: U2.6 (CLK), U3.52 (QSPI_SCLK)
- new net RST: SW4.2, U3.26 (RUN)
- new net SWCLK: U3.24 (SWCLK)
- new net SWDIO: U3.25 (SWD)
- new net TRIGGER: U3.11 (GPIO8), U6.3 (A)
- new net TRIGGER_IN: J9.1 (Pin_1), J9.2 (Pin_2), U6.4 (B)
- new net TRIGGER_VREF: J10.1 (Pin_1), J10.2 (Pin_2), U6.6 (VCCB)
- new net VBUS: D6.2 (A), F1.2, Q5.1 (G), R12.1
- new net VIN: C24.1, C5.1, SW2.2 (B), U1.1 (VIN), U1.3 (EN), U5.1 (IN), U5.3 (EN)
- new net VREF: J3.1 (Pin_1), SW7.4
- new net VREFOUT: C22.1, R15.1, SW7.3, U4.2 (VCCA)
- new net VSYS: D10.1 (K), Q5.3 (D)
- no-connect marks 0 -> 11
Other:
- note added: "DANGER: HIGH VOLTAGE"
- note added: "FLASH"
- note added: "Fault Injection"
- note added: "LEVEL SHIFTER"
- note added: "MOSFET Glitch"
- note added: "PIN CONNECTORS"
- note added: "TRIGGER LEVEL SHIFTER"
- note added: "Voltage Selector"
- title: (none) -> PicoFault

Commit message: Minor touch-ups
Parts:
- removed F1: 0.5A, Fuse:Fuse_0805_2012Metric, symbol Device:Fuse_Small
- removed P1: USB_C_Plug_USB2.0, Connectors:C393939, symbol Connector:USB_C_Plug_USB2.0
- removed R2, R4: 5.1K, Resistor_SMD:R_0603_1608Metric, symbol Device:R
- removed U3: RP2040, BuggyCat:RP2040-QFN-56, symbol PicoWAN-rescue:RP2040-MCU_RaspberryPi_and_Boards-PicoWAN-rescue-PicoWAN-rescue
- added F2: 0.5A, Fuse:Fuse_0805_2012Metric, symbol Device:Fuse_Small
- added R22, R27: 5.1K, Resistor_SMD:R_0603_1608Metric, symbol Device:R
- added U3: GT-USB-7010AN, PicoFault:USB-SMD_GT-USB-7010AN, symbol PicoFault:GT-USB-7010AN
- added U7: RP2040, PicoFault:LQFN-56_L7.0-W7.0-P0.4-EP, symbol PicoFault:RP2040
Connections:
- net +: now also U7.47 (USB_DP)
- net +1V2: now also U7.23 (DVDD), U7.45 (VREG_VOUT), U7.50 (DVDD)
- net +3V3: now also U7.1 (IOVDD), U7.10 (IOVDD), U7.22 (IOVDD), U7.33 (IOVDD), U7.42 (IOVDD), U7.43 (ADC_AVDD), U7.44 (VREG_IN), U7.48 (USB_VDD), U7.49 (IOVDD)
- net -: now also U7.46 (USB_DM)
- net ANALOG: now also U7.41 (GPIO29_ADC3)
- net CHARGED: now also U7.29 (GPIO18), U7.38 (GPIO26_ADC0)
- net D+: now also U3.A6 (DP1), U3.B6 (DP2)
- net D-: now also U3.A7 (DN1), U3.B7 (DN2)
- net GND: now also F2.2, R22.2, R27.2, U3.13 (GND), U3.14 (GND), U3.15 (GND), U3.16 (GND), U3.A1B12 (GND), U3.B1A12 (GND), U7.19 (TESTEN), U7.57 (GND)
- net GP0: now also U7.2 (GPIO0)
- net GP1: now also U7.3 (GPIO1)
- net GP10: now also U7.13 (GPIO10)
- net GP11: now also U7.14 (GPIO11)
- net GP2: now also U7.4 (GPIO2)
- net GP27: now also U7.39 (GPIO27_ADC1)
- net GP28: now also U7.40 (GPIO28_ADC2)
- net GP3: now also U7.5 (GPIO3)
- net GP4: now also U7.6 (GPIO4)
- net GP5: now also U7.7 (GPIO5)
- net GP6: now also U7.8 (GPIO6)
- net GP7: now also U7.9 (GPIO7)
- net GP9: now also U7.12 (GPIO9)
- net HPGLITCH2: now also U7.27 (GPIO16)
- net HVPULSE: now also U7.17 (GPIO14)
- net HVPWM: now also U7.31 (GPIO20)
- net LPGLITCH2: now also U7.28 (GPIO17)
- net QSPI_CS: now also U7.56 (QSPI_SS)
- net QSPI_DATA0: now also U7.53 (QSPI_SD0)
- net QSPI_DATA1: now also U7.55 (QSPI_SD1)
- net QSPI_DATA2: now also U7.54 (QSPI_SD2)
- net QSPI_DATA3: now also U7.51 (QSPI_SD3)
- net QSPI_SCK: now also U7.52 (QSPI_SCLK)
- net RST: now also U7.26 (RUN)
- net SWCLK: now also U7.24 (SWCLK)
- net SWDIO: now also U7.25 (SWD)
- net TRIGGER: now also U7.11 (GPIO8)
- net VBUS: now also F2.1, U3.A4B9 (VBUS), U3.B4A9 (VBUS)
- net at C8.1, Y1.1: now also U7.20 (XIN)
- net at R18.2: now also U7.21 (XOUT)
- new net: R27.1, U3.B5 (CC2)
- new net: R22.1, U3.A5 (CC1)
- no-connect marks 11 -> 13
Other:
- moved on the sheet: C2, D10, D2, D8, D9, J1, J6, R1, R12, R14, R16, R5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
